File: hardware/card.brd (EAGLE design)
At the start: 100 x 100 mm, 90 parts, among them J1 UE27AC54100, J2 B2PS-VH(LF)(SN), J3 MINI-USB-UX60A-MB-5ST, J4 MICROSD, J5 JST_2PIN, J6 0541323062, J7 JST_2PIN, J8 6-PIN_2MM-V, U1 ATSAMD21J_QFN, U2 MCP73833, U3 TLV70233DBVR, U4 ATWINC1500_MR210PA, U6 MIC2288YD5-TR, U7 TS3USB221, X3 32.768

Commit message: routing
Parts:
- removed U6: MIC2288YD5-TR, CardReader:TSOT-23-5
- removed U7: TS3USB221, CardReader:10-PIN-UQFN
- added C33: 1uF, rcl:C0603
- added U5: TLV70233DBVR, lib-card:SOT-23-5
- added X2: 32.768, lib-card:XTAL3215
- C1, C16, C2, C25: value 1uF -> 0.1uF
- C10, C8: value 1uF -> 22pF
- C14, C15: value 10uF -> 0.1uF
- C19, C30, C32, C9: value 0.1uF -> 1uF
- C23, C24: value 10uF -> 1uF
- C26, C27: value 1uF -> 10uF
- C28, C29: value 0.1uF -> 10uF
- C3: value 10uF -> 1uF; device rcl:C0805 -> rcl:C0603
- C6: value 22pF -> 0.1uF
- C7: value 22pF -> 10uF; device rcl:C0603 -> rcl:C0805
- D1, D11: value GREEN -> RED; device lib-card:CHIP-LED0603 -> RoboJackets-LEDs:CHIP-LED0603
- D10, D2, D9: device lib-card:CHIP-LED0603 -> RoboJackets-LEDs:CHIP-LED0603
- D3, D8: value RED -> GREEN; device lib-card:CHIP-LED0603 -> RoboJackets-LEDs:CHIP-LED0603
- D4: value YELLOW -> PMEG4010EGWX; device led:SMARTLED-TTW -> CardReader:SOD123
- D5: device led:SMARTLED-TTW -> RoboJackets-LEDs:CHIP-LED0603
- D6: value PMEG4010EGWX -> GREEN; device CardReader:SOD123 -> RoboJackets-LEDs:CHIP-LED0603
- D7: value RED -> GREEN; device led:SMARTLED-TTW -> RoboJackets-LEDs:CHIP-LED0603
- F1: value 2A -> 500mA
- F2: value 500mA -> 2A
- J2: value B2PS-VH(LF)(SN) -> MICROSD; device RoboJackets-Connectors:B2PS-CENTERED -> CardReader:MICROSD
- J3: value MINI-USB-UX60A-MB-5ST -> 0541323062; device lib-card:UX60A-MB-5ST -> CardReader:0541323062
- J4: value MICROSD -> 6-PIN_2MM-V; device CardReader:MICROSD -> RoboJackets-Connectors:2MM-6-V
- J6: value 0541323062 -> B2PS-VH(LF)(SN); device CardReader:0541323062 -> RoboJackets-Connectors:B2PS-CENTERED
- J7: value JST_2PIN -> MINI-USB-UX60A-MB-5ST; device card:JSTPH2 -> lib-card:UX60A-MB-5ST
- J8: value 6-PIN_2MM-V -> JST_2PIN; device RoboJackets-Connectors:2MM-6-V -> card:JSTPH2
- R1: value 330 -> 10k
- R10, R9: value 100k -> 1k; device RoboJackets-Resistors:R0603W -> rcl:R0603
- R11, R12, R19: device RoboJackets-Resistors:R0603W -> rcl:R0603
- R13: value 0 -> 5.62k 1%
- R14: value 5.62k 1% -> 1.87k 1%
- R15: value 1.87k 1% -> 10k 1%
- R16: value 0 -> 10k 1%; device RoboJackets-Resistors:R0603W -> rcl:R0603
- R17: value 2.2k -> 330; device RoboJackets-Resistors:R0603W -> rcl:R0603
- R18: value 100k -> 330; device RoboJackets-Resistors:R0603W -> rcl:R0603
- R2: value 330 -> 100k
- R21, R4: value 1k -> 0
- R22: value 1k -> 10k
- R23: value 1k -> 330
- R3: value 330 -> 2.2k
- R5: value 10k -> 100k
- R6: value 10k 1% -> 1k
- R7: value 10k -> 1k
- R8: value 10k 1% -> 100k
- S2: value TL1000F160Q -> KAE01SGGT; device CardReader:TL1100 -> CardReader:KAE01SGGT
- S6: value KAE01SGGT -> TL1000F160Q; device CardReader:KAE01SGGT -> CardReader:TL1100
- U2: value MCP73833 -> TS3USB221; device CardReader:MSOP10 -> CardReader:10-PIN-UQFN
- U3: value TLV70233DBVR -> MIC2288YD5-TR; device lib-card:SOT-23-5 -> CardReader:TSOT-23-5
- U4: value ATWINC1500_MR210PA -> MCP73833; device CardReader:ATWINC1500_MR210PA -> CardReader:MSOP10
- X3: value 32.768 -> ATWINC1500_MR210PA; device lib-card:XTAL3215 -> CardReader:ATWINC1500_MR210PA
- moved S2 98.6 mm to (27.5, 5.00), turned to 90 degrees
- moved C21 93.6 mm to (80.5, 16.0), turned to 90 degrees
- moved C22 93.3 mm to (74.2, 9.50)
- moved S5 89.2 mm to (13.0, 31.5), flipped to the bottom
- moved J2 87.9 mm to (82.2, 21.8), flipped to the top, turned to 0 degrees
- moved J4 81.7 mm to (89.2, 29.0), flipped to the top, turned to 180 degrees
- moved R4 79.8 mm to (92.0, 18.0), turned to 90 degrees
- moved D6 79.1 mm to (92.8, 33.8)
- moved R9 78.4 mm to (86.2, 32.5), turned to 90 degrees
- moved J8 77.6 mm to (91.0, 9.00), flipped to the bottom, turned to 180 degrees
- moved C23 76.3 mm to (75.8, 13.0)
- moved C25 72.7 mm to (70.8, 16.0)
- moved R11 72.4 mm to (89.5, 32.5), turned to 90 degrees
- moved J3 71.9 mm to (75.0, 11.0), flipped to the bottom
- moved C24 71.3 mm to (74.2, 16.0), flipped to the bottom, turned to 90 degrees
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Connections:
- net !RESET: now also C6.1
- net +3.3V: now also C1.1, C11.1, C2.1, C25.1, C3.1, C33.1, C9.1, D2.A, D3.A, J2.4, J3.22, J3.4, J3.5, J4.3, J8.1, R10.1, U2.10, U5.5, X3.J10, X3.J20, X3.J23; no longer C16.1, C21.1, C22.1, C29.1, C30.1, C31.1, C32.1, D4.A@1, D5.A@1, J4.4, J6.26, J6.27, J6.9, J7.1, J8.3, R21.1, U3.5, U4.J10, U4.J20, U4.J23, U7.10
- net +5V: now also C31.1, C7.1, D10.A, D11.A, D9.A, J4.5, J7.1, R9.1, U4.1, U4.2; no longer C26.1, C3.1, D1.A, D2.A, D3.A, J3.1, J8.5, R20.1, U2.1, U2.2
- net 1D+: now also J7.3, U2.1; no longer J3.3, U7.1
- net 1D-: now also J7.2, U2.2; no longer J3.2, U7.2
- net 2D+: now also U2.3; no longer U7.3
- net 2D-: now also U2.4; no longer U7.4
- net 3V3_EN: now also R19.1, U5.3; no longer R7.1, U3.3
- net BATT: now also C32.2, F2.1, J6.2, R21.1, U4.10, U4.9; no longer C27.2, F1.1, J2.2, R13.1, U2.10, U2.9
- net BATT-MONITOR: now also R15.2, R16.1; no longer R6.2, R8.1
- net BATT-PRE-FUSE: now also F2.2; no longer F1.2
- net BOOST_FB: now also R13.1, R14.2, U3.3; no longer R14.1, R15.2, U6.3
- net BOOST_OUTPUT: now also C27.1, C28.1, C29.1, D4.C, F1.1, R13.2; no longer C15.1, C23.1, C24.1, D6.C, F2.1, R14.2
- net BOOST_SW: now also D4.A, U3.1; no longer D6.A, U6.1
- net BTN-DOWN: now also C13.1, S4.1, U1.3; no longer C18.1, S3.1, S3.2, U1.28
- net BTN-LEFT: now also C14.1, S5.1, U1.7; no longer C19.1, S4.1, S4.2, U1.25
- net BTN-RIGHT: now also C15.1, S6.2, U1.8; no longer C20.1, S5.1, S5.2, U1.24
- net BTN-UP: now also C12.1, S3.1, U1.10; no longer C17.1, S2.1, S2.2, U1.27
- net CHRG-!PG: now also R23.1, U4.7; no longer R3.1, U2.7
- net CHRG-PROG: now also R20.2, U4.6; no longer R4.2, U2.6
- net CHRG-STAT1: now also R18.1, U4.3; no longer R2.1, U2.3
- net CHRG-STAT2: now also R17.1, U4.4; no longer R1.1, U2.4
- net CHRG-THERM: now also R22.2, U4.8; no longer R5.2, U2.8
- net D+: now also U2.8; no longer U7.8
- net D-: now also U2.7; no longer U7.7
- net GND: now also C1.2, C2.2, C27.2, C32.1, C33.2, C8.2, D1.C, D5.C, D6.C, D7.C, J2.6, J2.MT1, J2.MT2, J3.10, J3.11, J3.14, J3.21, J3.29, J3.30, J3.6, J3.7, J3.8, J3.9, J4.1, J7.5, R14.1, R2.1, R20.1, R22.1, R4.2, R5.2, R8.1, S2.2, S6.3, S6.4, U2.6, U4.5, U5.2, X3.J12, X3.J28, X3.J9; no longer C19.2, C22.2, C23.2, C27.1, C32.2, D10.C, D11.C, D7.C@1, D9.C, J3.5, J4.6, J4.MT1, J4.MT2, J6.1, J6.10, J6.17, J6.2, J6.20, J6.21, J6.22, J6.23, J6.24, J6.25, J8.1, R10.2, R15.1, R18.1, R4.1, R5.1, R8.2, R9.1, S2.3, S2.4, S6.2, U4.J12, U4.J28, U4.J9, U6.2, U7.5, U7.6
- net LCD-!CS: now also J3.1, U1.23; no longer J6.30, U1.29
- net LCD-!RES: now also J3.2, U1.24; no longer J6.29, U1.31
- net LCD-A0: now also J3.3, U1.25; no longer J6.28, U1.48
- net LCD-CA1+: now also C22.1, J3.18; no longer C2.1, J6.13
- net LCD-CA1-: now also C22.2, C23.2, J3.17; no longer C1.2, C2.2, J6.14
- net LCD-CA2+: now also C19.1, J3.19; no longer C8.1, J6.12
- net LCD-CA2-: now also C19.2, J3.20; no longer C8.2, J6.11
- net LCD-CA3+: now also C23.1, J3.16; no longer C1.1, J6.15
- net LCD-K: now also J8.2, R4.1; no longer J7.2, R16.1
- net LCD-MOSI: now also J3.13; no longer J6.18
- net LCD-SCK: now also J3.12; no longer J6.19
- net LCD-V0: now also C18.1, J3.27; no longer C28.1, J6.4
- net LCD-V1: now also C21.1, J3.26; no longer C13.1, J6.5
- net LCD-V2: now also C17.1, J3.25; no longer C12.1, J6.6
- net LCD-V3: now also C20.1, J3.24; no longer C11.1, J6.7
- net LCD-V4: now also C16.1, J3.23; no longer C9.1, J6.8
- net LCD-VOUT: now also C24.1, J3.15; no longer C10.1, J6.16
- net LED-!PG: now also D11.C, R23.2; no longer D3.C, R3.2
- net LED-3V3: now also D6.A, R10.2; no longer D9.A, R21.2
- net LED-5V: now also D8.A, R12.2; no longer D11.A, R23.2
- net LED-STAT1: now also D10.C, R18.2; no longer D2.C, R2.2
- net LED-STAT2: now also D9.C, R17.2; no longer D1.C, R1.2
- net LED-VBATT: now also D7.A, R11.2; no longer D10.A, R22.2
- net LED-VBUS: now also D5.A, R9.2; no longer D8.A, R20.2
- net MISO: now also J2.7, X3.J17; no longer J4.7, U4.J17
- net MOSI: now also J2.3, X3.J15; no longer J4.3, U4.J15
- net PROG-LED: now also D1.A, R3.2; no longer D7.A@1, R17.2
- net PROG-LED-2: now also R3.1; no longer R17.1
- net SCK: now also J2.5, X3.J18; no longer J4.5, U4.J18
- net SD-!CD: now also J2.CD1, U1.16; no longer J4.CD1, U1.14
- net SD-!CS: now also J2.2, U1.27; no longer J4.2, U1.12
- net USB-HOST-EN: now also R1.1; no longer R19.1
- net USB-S: now also R1.2, R2.2, S2.1, U2.9; no longer R18.2, R19.2, S6.1, U7.9
- net VBATT: now also C26.1, C30.1, J4.4, J6.1, R11.1, R15.1, R19.2, R21.2, U3.4, U3.5, U5.1; no longer C14.1, C25.1, J2.1, J8.4, R13.2, R22.1, R6.1, R7.2, U3.1, U6.4, U6.5
- net VBUS: now also F1.2, J4.6, R12.1; no longer F2.2, J8.6, R23.1
- net WIFI-!CS: now also X3.J16; no longer U4.J16
- net WIFI-!IRQ: now also U1.14, X3.J13; no longer U1.30, U4.J13
- net WIFI-!RESET: now also R8.2, X3.J4; no longer R9.2, U4.J4
- net WIFI-CHIP-EN: now also R5.1, U1.12, X3.J22; no longer R10.1, U1.23, U4.J22
- net WIFI-GPIO15: now also R7.2, X3.J26; no longer R12.2, U4.J26
- net WIFI-GPIO16: now also R6.1, X3.J27; no longer R11.1, U4.J27
- net WIFI-LED-G: now also D3.C, R7.1; no longer D5.C@1, R12.1
- net WIFI-LED-Y: now also D2.C, R6.2; no longer D4.C@1, R11.2
- net WIFI-WAKE: now also X3.J11; no longer U4.J11
- net X3-1: now also C8.1, X2.P$1; no longer C6.1, X3.P$1
- net X3-2: now also C10.1, X2.P$2; no longer C7.1, X3.P$2
Routing:
- net +3.3V: track 82.3 -> 151.5 mm, vias 5 -> 14
- net +5V: track 67.9 -> 131.4 mm
- net BTN-LEFT: track 1.48 -> 64.5 mm, vias 1 -> 0
- net USB-S: track 8.69 -> 68.5 mm, vias 0 -> 4
- net WIFI-!IRQ: track 77.6 -> 17.9 mm, vias 3 -> 2
- net GND: track 75.2 -> 16.9 mm, vias 22 -> 11
- net BTN-UP: track 3.98 -> 60.2 mm, vias 1 -> 4
- net !RESET: track 14.3 -> 70.5 mm, vias 1 -> 4
- net WIFI-CHIP-EN: track 73.9 -> 19.4 mm, vias 1 -> 2
- net BTN-RIGHT: track 2.19 -> 52.4 mm, vias 1 -> 0
- net BTN-DOWN: track 3.02 -> 51.9 mm, vias 1 -> 0
- net VBUS: track 3.15 -> 40.2 mm
- net MOSI: track 6.57 -> 42.8 mm, vias 1 -> 4
- net SCK: track 6.98 -> 38.1 mm, vias 1 -> 2
- net MISO: track 6.57 -> 37.1 mm, vias 1 -> 2
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- added copper zone on layer 1, net GND
Other:
- board size 100 x 100 mm -> 97 x 56 mm
- board text added: "+3.3V"
- board text added: "+5V"
- board text added: "VBAT"
- board text added: "VBUS"
