File: hardware/card.sch (EAGLE design)
At the start: 90 parts, among them J1 UE27AC54100, J2 B2PS-VH(LF)(SN), J3 MINI-USB-UX60A-MB-5ST, J4 MICROSD, J5 JST_2PIN, J6 0541323062, J7 JST_2PIN, J8 6-PIN_2MM-V, U1 ATSAMD21J_QFN, U2 MCP73833, U3 TLV70233DBVR, U4 ATWINC1500_MR210PA, U6 MIC2288YD5-TR, U7 TS3USB221, X3 32.768

Commit message: routing
Parts:
- removed U6: MIC2288YD5-TR, CardReader:MIC2288YD5-TR
- removed U7: TS3USB221, CardReader:TS3USB221
- added C33: 1uF, rcl:C-USC0603
- added U5: TLV70233DBVR, lib-card:TLV70233DBVR
- added X2: 32.768, lib-card:XTAL-3.2X1.5
- C1, C16, C2, C25: value 1uF -> 0.1uF
- C10, C8: value 1uF -> 22pF
- C14, C15: value 10uF -> 0.1uF
- C19, C30, C32, C9: value 0.1uF -> 1uF
- C23, C24: value 10uF -> 1uF
- C26, C27: value 1uF -> 10uF
- C28, C29: value 0.1uF -> 10uF
- C3: value 10uF -> 1uF; device rcl:C-USC0805 -> rcl:C-USC0603
- C6: value 22pF -> 0.1uF
- C7: value 22pF -> 10uF; device rcl:C-USC0603 -> rcl:C-USC0805
- D1, D11: value GREEN -> RED; device lib-card:LED-SMD-GREEN -> RoboJackets-LEDs:LED-SMD-RED
- D10: device lib-card:LED-SMD-GREEN -> RoboJackets-LEDs:LED-SMD-YELLOW
- D2: device lib-card:LED-SMD-YELLOW -> RoboJackets-LEDs:LED-SMD-YELLOW
- D3: value RED -> GREEN; device lib-card:LED-SMD-RED -> RoboJackets-LEDs:LED-SMD-GREEN
- D4: value YELLOW -> PMEG4010EGWX; device led:LED -> CardReader:SCHOTTKEY-DIODE-SOD123
- D5: device led:LED -> RoboJackets-LEDs:LED-SMD-GREEN
- D6: value PMEG4010EGWX -> GREEN; device CardReader:SCHOTTKEY-DIODE-SOD123 -> RoboJackets-LEDs:LED-SMD-GREEN
- D7: value RED -> GREEN; device led:LED -> RoboJackets-LEDs:LED-SMD-GREEN
- D8: value RED -> GREEN; device lib-card:LED-SMD-GREEN -> RoboJackets-LEDs:LED-SMD-GREEN
- D9: device lib-card:LED-SMD-GREEN -> RoboJackets-LEDs:LED-SMD-GREEN
- F1: value 2A -> 500mA
- F2: value 500mA -> 2A
- J2: value B2PS-VH(LF)(SN) -> MICROSD; device RoboJackets-Connectors:B2PS-VH(LF)(SN) -> CardReader:MICROSD
- J3: value MINI-USB-UX60A-MB-5ST -> 0541323062; device lib-card:MINI-USB-UX60A-MB-5ST -> CardReader:0541323062
- J4: value MICROSD -> 6-PIN_2MM-V; device CardReader:MICROSD -> RoboJackets-Connectors:6-PIN_2MM-V
- J6: value 0541323062 -> B2PS-VH(LF)(SN); device CardReader:0541323062 -> RoboJackets-Connectors:B2PS-VH(LF)(SN)
- J7: value JST_2PIN -> MINI-USB-UX60A-MB-5ST; device card:JST_2PIN -> lib-card:MINI-USB-UX60A-MB-5ST
- J8: value 6-PIN_2MM-V -> JST_2PIN; device RoboJackets-Connectors:6-PIN_2MM-V -> card:JST_2PIN
- R1: value 330 -> 10k
- R10, R9: value 100k -> 1k; device RoboJackets-Resistors:R0603W -> rcl:R-US_R0603
- R11, R12, R19: device RoboJackets-Resistors:R0603W -> rcl:R-US_R0603
- R13: value 0 -> 5.62k 1%
- R14: value 5.62k 1% -> 1.87k 1%
- R15: value 1.87k 1% -> 10k 1%
- R16: value 0 -> 10k 1%; device RoboJackets-Resistors:R0603W -> rcl:R-US_R0603
- R17: value 2.2k -> 330; device RoboJackets-Resistors:R0603W -> rcl:R-US_R0603
- R18: value 100k -> 330; device RoboJackets-Resistors:R0603W -> rcl:R-US_R0603
- R2: value 330 -> 100k
- R21, R4: value 1k -> 0
- R22: value 1k -> 10k
- R23: value 1k -> 330
- R3: value 330 -> 2.2k
- R5: value 10k -> 100k
- R6: value 10k 1% -> 1k
- R7: value 10k -> 1k
- R8: value 10k 1% -> 100k
- S2: value TL1000F160Q -> KAE01SGGT; device CardReader:TL1000F160Q -> CardReader:KAE01SGGT
- S6: value KAE01SGGT -> TL1000F160Q; device CardReader:KAE01SGGT -> CardReader:TL1000F160Q
- U2: value MCP73833 -> TS3USB221; device CardReader:MCP73833 -> CardReader:TS3USB221
- U3: value TLV70233DBVR -> MIC2288YD5-TR; device lib-card:TLV70233DBVR -> CardReader:MIC2288YD5-TR
- U4: value ATWINC1500_MR210PA -> MCP73833; device CardReader:ATWINC1500_MR210PA -> CardReader:MCP73833
- X3: value 32.768 -> ATWINC1500_MR210PA; device lib-card:XTAL-3.2X1.5 -> CardReader:ATWINC1500_MR210PA
Connections:
- net !RESET: now also C6.1
- net +3.3V: now also C1.1, C11.1, C2.1, C25.1, C3.1, C33.1, C9.1, D2.A, D3.A, J2.VDD, J3.22, J3.4, J3.5, J4.3, J8.1, R10.1, U2.VCC, U5.VOUT, X3.SPI_CFG, X3.VBAT, X3.VDDIO; no longer C16.1, C21.1, C22.1, C29.1, C30.1, C31.1, C32.1, D4.A, D5.A, J4.VDD, J6.22, J6.4, J6.5, J7.1, J8.3, R21.1, U3.VOUT, U4.SPI_CFG, U4.VBAT, U4.VDDIO, U7.VCC
- net +5V: now also C31.1, C7.1, D10.A, D11.A, D9.A, J4.5, J7.1, R9.1, U4.VDD1, U4.VDD2; no longer C26.1, C3.1, D1.A, D2.A, D3.A, J3.1, J8.5, R20.1, U2.VDD1, U2.VDD2
- net 1D+: now also J7.3, U2.1D+; no longer J3.3, U7.1D+
- net 1D-: now also J7.2, U2.1D-; no longer J3.2, U7.1D-
- net 2D+: now also U2.2D+; no longer U7.2D+
- net 2D-: now also U2.2D-; no longer U7.2D-
- net 3V3_EN: now also R19.1, U5.EN; no longer R7.1, U3.EN
- net BATT: now also C32.2, F2.1, J6.2, R21.1, U4.VBAT1, U4.VBAT2; no longer C27.2, F1.1, J2.2, R13.1, U2.VBAT1, U2.VBAT2
- net BATT-MONITOR: now also R15.2, R16.1; no longer R6.2, R8.1
- net BATT-PRE-FUSE: now also F2.2; no longer F1.2
- net BOOST_FB: now also R13.1, R14.2, U3.FB; no longer R14.1, R15.2, U6.FB
- net BOOST_OUTPUT: now also C27.1, C28.1, C29.1, D4.C, F1.1, R13.2; no longer C15.1, C23.1, C24.1, D6.C, F2.1, R14.2
- net BOOST_SW: now also D4.A, U3.SW; no longer D6.A, U6.SW
- net BTN-DOWN: now also C13.1, S4.1A, U1.PA02/EINT2/AIN0/Y0/VOUT; no longer C18.1, S3.1, U1.PA19/I3/SERCOM1+3.3/I2SD0
- net BTN-LEFT: now also C14.1, S5.1A, U1.PB08/I8/AIN2/SERCOM4.0; no longer C19.1, S4.1, U1.PA16/I2C/I0/SERCOM1+3.0
- net BTN-RIGHT: now also C15.1, S6.1B, U1.PB09/I9/AIN3/SERCOM4.1; no longer C20.1, S5.1, U1.PA15/I15/SERCOM3+4.3
- net BTN-UP: now also C12.1, S3.1A, U1.PA05/EINT5/AIN5/SERCOM0.1; no longer C17.1, S2.1, U1.PA18/I2/SERCOM1+3.2
- net CHRG-!PG: now also R23.1, U4.PG; no longer R3.1, U2.PG
- net CHRG-PROG: now also R20.2, U4.PROG; no longer R4.2, U2.PROG
- net CHRG-STAT1: now also R18.1, U4.STAT1; no longer R2.1, U2.STAT1
- net CHRG-STAT2: now also R17.1, U4.STAT2; no longer R1.1, U2.STAT2
- net CHRG-THERM: now also R22.2, U4.THERM; no longer R5.2, U2.THERM
- net D+: now also U2.D+; no longer U7.D+
- net D-: now also U2.D-; no longer U7.D-
- net GND: now also C1.2, C2.2, C27.2, C32.1, C33.2, C8.2, D1.K, D5.K, D6.K, D7.K, J2.GND, J2.GND1, J2.VSS, J3.10, J3.11, J3.14, J3.21, J3.29, J3.30, J3.6, J3.7, J3.8, J3.9, J4.1, J7.5, R14.1, R16.2, R2.1, R20.1, R22.1, R4.2, R5.2, R8.1, S3.2A, S3.2B, S4.2A, S4.2B, S5.2A, S5.2B, S6.2A, S6.2B, U2.OE, U5.GND, X3.GND, X3.GND@1, X3.GND@2; no longer C19.2, C22.2, C23.2, C27.1, C32.2, D10.K, D11.K, D7.C, D9.K, J3.5, J4.GND, J4.GND1, J4.VSS, J6.10, J6.11, J6.14, J6.21, J6.29, J6.30, J6.6, J6.7, J6.8, J6.9, J8.1, R10.PIN2, R15.1, R16.PIN2, R18.PIN1, R4.1, R5.1, R8.2, R9.PIN1, S3.2, S4.2, S5.2, S6.2, U4.GND@1, U4.GND@2, U6.GND, U7.GND, U7.OE
- net LCD-!CS: now also J3.1, U1.PA14/I14/SERCOM2+4.2; no longer J6.1, U1.PA20/I4/SERCOM3+5.2/I2SSC
- net LCD-!RES: now also J3.2, U1.PA15/I15/SERCOM3+4.3; no longer J6.2, U1.PA22/I2C/I6/SERCOM3+5.0
- net LCD-A0: now also J3.3, U1.PA16/I2C/I0/SERCOM1+3.0; no longer J6.3, U1.PB03/I3/AIN11/SERCOM5.1
- net LCD-CA1+: now also C22.1, J3.18; no longer C2.1, J6.18
- net LCD-CA1-: now also C22.2, C23.2, J3.17; no longer C1.2, C2.2, J6.17
- net LCD-CA2+: now also C19.1, J3.19; no longer C8.1, J6.19
- net LCD-CA2-: now also C19.2, J3.20; no longer C8.2, J6.20
- net LCD-CA3+: now also C23.1, J3.16; no longer C1.1, J6.16
- net LCD-K: now also J8.2, R4.1; no longer J7.2, R16.PIN1
- net LCD-MOSI: now also J3.13; no longer J6.13
- net LCD-SCK: now also J3.12; no longer J6.12
- net LCD-V0: now also C18.1, J3.27; no longer C28.1, J6.27
- net LCD-V1: now also C21.1, J3.26; no longer C13.1, J6.26
- net LCD-V2: now also C17.1, J3.25; no longer C12.1, J6.25
- net LCD-V3: now also C20.1, J3.24; no longer C11.1, J6.24
- net LCD-V4: now also C16.1, J3.23; no longer C9.1, J6.23
- net LCD-VOUT: now also C24.1, J3.15; no longer C10.1, J6.15
- net LED-!PG: now also D11.K, R23.2; no longer D3.K, R3.2
- net LED-3V3: now also D6.A, R10.2; no longer D9.A, R21.2
- net LED-5V: now also D8.A, R12.2; no longer D11.A, R23.2
- net LED-STAT1: now also D10.K, R18.2; no longer D2.K, R2.2
- net LED-STAT2: now also D9.K, R17.2; no longer D1.K, R1.2
- net LED-VBATT: now also D7.A, R11.2; no longer D10.A, R22.2
- net LED-VBUS: now also D5.A, R9.2; no longer D8.A, R20.2
- net MISO: now also J2.DATA_OUT, X3.MISO; no longer J4.DATA_OUT, U4.MISO
- net MOSI: now also J2.DATA_IN, X3.MOSI; no longer J4.DATA_IN, U4.MOSI
- net PROG-LED: now also D1.A, R3.2; no longer D7.A, R17.PIN2
- net PROG-LED-2: now also R3.1; no longer R17.PIN1
- net SCK: now also J2.SCLK, X3.SCK; no longer J4.SCLK, U4.SCK
- net SD-!CD: now also J2.CARD_DETECT, U1.PA11/I11/AIN19/SERCOM0+2.3/I2SF0; no longer J4.CARD_DETECT, U1.PA09/I2C/I9/AIN17/SERCOM0+2.1/I2SMC
- net SD-!CS: now also J2.CS, U1.PA18/I2/SERCOM1+3.2; no longer J4.CS, U1.PA07/I7/AIN7/SERCOM0.3/I2SD0
- net USB-HOST-EN: now also R1.1; no longer R19.PIN1
- net USB-S: now also R1.2, R2.2, S2.1, U2.S; no longer R18.PIN2, R19.PIN2, S6.1, U7.S
- net VBATT: now also C26.1, C30.1, J4.4, J6.1, R11.1, R15.1, R19.2, R21.2, U3.EN, U5.VIN; no longer C14.1, C25.1, J2.1, J8.4, R13.2, R22.1, R6.1, R7.2, U6.EN, U6.VIN
- net VBUS: now also F1.2, J4.6, R12.1; no longer F2.2, J8.6, R23.1
- net WIFI-!CS: now also X3.CS; no longer U4.CS
- net WIFI-!IRQ: now also U1.PA09/I2C/I9/AIN17/SERCOM0+2.1/I2SMC, X3.!IRQ; no longer U1.PA21/I5/SERCOM3+5.3/I2SFS0, U4.!IRQ
- net WIFI-!RESET: now also R8.2, X3.!RESET; no longer R9.PIN2, U4.!RESET
- net WIFI-CHIP-EN: now also R5.1, U1.PA07/I7/AIN7/SERCOM0.3/I2SD0, X3.CHIP_EN; no longer R10.PIN1, U1.PA14/I14/SERCOM2+4.2, U4.CHIP_EN
- net WIFI-GPIO15: now also R7.2, X3.GPIO15; no longer R12.PIN2, U4.GPIO15
- net WIFI-GPIO16: now also R6.1, X3.GPIO16; no longer R11.PIN1, U4.GPIO16
- net WIFI-LED-G: now also D3.K, R7.1; no longer D5.C, R12.PIN1
- net WIFI-LED-Y: now also D2.K, R6.2; no longer D4.C, R11.PIN2
- net WIFI-WAKE: now also X3.WAKE; no longer U4.WAKE
- net X3-1: now also C8.1, X2.P$1; no longer C6.1, X3.P$1
- net X3-2: now also C10.1, X2.P$2; no longer C7.1, X3.P$2
